File: sense2.0/Hardware/Rele-board.brd (EAGLE design)
At the start: 158.1 x 100 mm, 23 parts, among them K1 5Vcc, K2 5Vcc, Q1 BC338, Q2 BC338

Commit message: As built
Parts:
- removed MOD1: ESP12E_DEVKIT, ESP12E_DEVKIT:ESP12E_DEVKIT
- added JP2, JP3: (no value), pinhead:1X15
- moved H2 7.62 mm to (14.6, 95.2)
- moved H3 7.62 mm to (78.7, 95.2)
Connections:
- net GND: now also JP2.10, JP3.14; no longer MOD1.GND@0, MOD1.GND@3
- net N$2: now also JP2.15; no longer MOD1.VIN
- net RELE_1_IO: now also JP3.4; no longer MOD1.D3
- net RELE_2_IO: now also JP3.5; no longer MOD1.D4
Routing:
- net RELE_1_IO: track 35.4 -> 48.9 mm
- net RELE_2_IO: track 51.2 -> 64.6 mm
- net N$2: track 9.99 -> 13.2 mm
Other:
- board size 158.1 x 100 mm -> 70.5 x 95.6 mm
