File: sense2.0/Hardware/Rele-board.sch (EAGLE design)
At the start: 23 parts, among them K1 5Vcc, K2 5Vcc, Q1 BC338, Q2 BC338

Commit message: As built
Parts:
- removed MOD1: ESP12E_DEVKIT, ESP12E_DEVKIT:ESP12E_DEVKIT
- added JP2, JP3: (no value), pinhead:PINHD-1X15
Connections:
- net GND: now also JP2.10, JP3.14; no longer MOD1.GND@0, MOD1.GND@3
- net N$2: now also JP2.15; no longer MOD1.VIN
- net RELE_1_IO: now also JP3.4; no longer MOD1.D3
- net RELE_2_IO: now also JP3.5; no longer MOD1.D4
Changed lines of the file:
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@@
 <?xml version="1.0" encoding="utf-8"?>
 <!DOCTYPE eagle SYSTEM "eagle.dtd">
-<eagle version="8.3.1">
+<eagle version="8.2.2">
 <drawing>
 <settings>
 <setting alwaysvectorfont="no"/>
-<setting keepoldvectorfont="yes"/>
 <setting verticaltext="up"/>
 </settings>
@@
 </classes>
 <parts>
-<part name="MOD1" library="ESP12E_DEVKIT" deviceset="ESP12E_DEVKIT" device=""/>
 <part name="FONTE" library="hlk-pm01" deviceset="HLK-PM01" device="">
 <attribute name="FONTE" value="127Vac - 5Vcc"/>
 </part>
-<part name="X2" library="con-ptr500" library_urn="urn:adsk.eagle:library:181" deviceset="AK300/2" device="" package3d_urn="urn:adsk.eagle:package:9881/1"/>
+<part name="X2" library="con-ptr500" library_urn="urn:adsk.eagle:library:181" deviceset="AK300/2" device=""/>
 <part name="GND5" library="supply1" deviceset="GND" device=""/>
 <part name="P+1" library="supply1" library_urn="urn:adsk.eagle:library:371" deviceset="+5V" device=""/>
@@
 <part name="C2" library="rcl" deviceset="CPOL-US" device="E2.5-6" value="0.1uF"/>
 <part name="GND1" library="supply1" deviceset="GND" device=""/>
-<part name="H1" library="special-drill" library_urn="urn:adsk.eagle:library:366" deviceset="SPECIAL_DRILL_" device="0.1000" package3d_urn="urn:adsk.eagle:package:26539/1"/>
-<part name="H2" library="special-drill" library_urn="urn:adsk.eagle:library:366" deviceset="SPECIAL_DRILL_" device="0.1000" package3d_urn="urn:adsk.eagle:package:26539/1"/>
-<part name="H3" library="special-drill" library_urn="urn:adsk.eagle:library:366" deviceset="SPECIAL_DRILL_" device="0.1000" package3d_urn="urn:adsk.eagle:package:26539/1"/>
-<part name="H4" library="special-drill" library_urn="urn:adsk.eagle:library:366" deviceset="SPECIAL_DRILL_" device="0.1000" package3d_urn="urn:adsk.eagle:package:26539/1"/>
+<part name="H1" library="special-drill" library_urn="urn:adsk.eagle:library:366" deviceset="SPECIAL_DRILL_" device="0.1000"/>
+<part name="H2" library="special-drill" library_urn="urn:adsk.eagle:library:366" deviceset="SPECIAL_DRILL_" device="0.1000"/>
+<part name="H3" library="special-drill" library_urn="urn:adsk.eagle:library:366" deviceset="SPECIAL_DRILL_" device="0.1000"/>
+<part name="H4" library="special-drill" library_urn="urn:adsk.eagle:library:366" deviceset="SPECIAL_DRILL_" device="0.1000"/>
 <part name="K1" library="relay" deviceset="CQ1-12V" device="" value="5Vcc"/>
 <part name="Q1" library="transistor-npn" deviceset="BC338*" device=""/>
@@
 <part name="P+2" library="supply1" library_urn="urn:adsk.eagle:library:371" deviceset="+5V" device=""/>
 <part name="P+3" library="supply1" library_urn="urn:adsk.eagle:library:371" deviceset="+5V" device=""/>
-<part name="X1" library="con-ptr500" library_urn="urn:adsk.eagle:library:181" deviceset="AK300/3" device="" package3d_urn="urn:adsk.eagle:package:9878/1"/>
-<part name="X5" library="con-ptr500" library_urn="urn:adsk.eagle:library:181" deviceset="AK300/3" device="" package3d_urn="urn:adsk.eagle:package:9878/1"/>
+<part name="X1" library="con-ptr500" library_urn="urn:adsk.eagle:library:181" deviceset="AK300/3" device=""/>
+<part name="X5" library="con-ptr500" library_urn="urn:adsk.eagle:library:181" deviceset="AK300/3" device=""/>
 <part name="GND2" library="supply1" deviceset="GND" device=""/>
 <part name="GND3" library="supply1" deviceset="GND" device=""/>
+<part name="JP2" library="pinhead" library_urn="urn:adsk.eagle:library:325" deviceset="PINHD-1X15" device=""/>
+<part name="JP3" library="pinhead" library_urn="urn:adsk.eagle:library:325" deviceset="PINHD-1X15" device=""/>
 </parts>
 <sheets>
@@
 </plain>
 <instances>
-<instance part="MOD1" gate="G$1" x="172.72" y="140.97"/>
 <instance part="FONTE" gate="G$1" x="66.802" y="158.75" rot="MR180">
 <attribute name="FONTE" x="74.422" y="163.576" size="1.778" layer="96" rot="MR180"/>
@@
 <instance part="GND2" gate="1" x="256.54" y="113.284"/>
 <instance part="GND3" gate="1" x="320.04" y="113.284"/>
+<instance part="JP2" gate="A" x="157.48" y="140.97"/>
+<instance part="JP3" gate="A" x="187.96" y="140.97" rot="MR0"/>
 </instances>
 <busses>
@@
 <net name="GND" class="0">
 <segment>
-<pinref part="MOD1" gate="G$1" pin="GND@3"/>
 <wire x1="190.5" y1="125.73" x2="196.85" y2="125.73" width="0.1524" layer="91"/>
 <pinref part="GND5" gate="1" pin="GND"/>
-</segment>
-<segment>
-<pinref part="MOD1" gate="G$1" pin="GND@0"/>
+<pinref part="JP3" gate="A" pin="14"/>
+</segment>
+<segment>
 <pinref part="GND1" gate="1" pin="GND"/>
 <wire x1="151.13" y1="135.89" x2="154.94" y2="135.89" width="0.1524" layer="91"/>
+<pinref part="JP2" gate="A" pin="10"/>
 </segment>
 <segment>
@@
 <net name="RELE_1_IO" class="0">
 <segment>
-<pinref part="MOD1" gate="G$1" pin="D3"/>
 <wire x1="190.5" y1="151.13" x2="195.58" y2="151.13" width="0.1524" layer="91"/>
 <label x="195.58" y="151.13" size="1.778" layer="95"/>
+<pinref part="JP3" gate="A" pin="4"/>
 </segment>
 <segment>
@@
 <net name="RELE_2_IO" class="0">
 <segment>
-<pinref part="MOD1" gate="G$1" pin="D4"/>
 <wire x1="190.5" y1="148.59" x2="195.58" y2="148.59" width="0.1524" layer="91"/>
 <label x="195.58" y="148.59" size="1.778" layer="95"/>
+<pinref part="JP3" gate="A" pin="5"/>
 </segment>
 <segment>
@@
 <net name="N$2" class="0">
 <segment>
-<pinref part="MOD1" gate="G$1" pin="VIN"/>
 <pinref part="JP1" gate="A" pin="1"/>
 <wire x1="150.114" y1="123.19" x2="154.94" y2="123.19" width="0.1524" layer="91"/>
+<pinref part="JP2" gate="A" pin="15"/>
 </segment>
 </net>
@@
 <compatibility>
 <note version="8.2" severity="warning">
-Since Version 8.2, EAGLE supports online libraries. The ids
+Since Version 8.2, Eagle supports online libraries. The ids
 of those online libraries will not be understood (or retained)
 with this version.
 </note>
-<note version="8.3" severity="warning">
-Since Version 8.3, EAGLE supports URNs for individual library
-assets (packages, symbols, and devices). The URNs of those assets
-will not be understood (or retained) with this version.
-</note>
-<note version="8.3" severity="warning">
-Since Version 8.3, EAGLE supports the association of 3D packages
-with devices in libraries, schematics, and board files. Those 3D
-packages will not be understood (or retained) with this version.
-</note>
 </compatibility>
