File: sense2.0/Hardware/TBD-board.brd (EAGLE design)
At the start: 160 x 100 mm, 17 parts, among them IC1 LM324N, X1 PG203J

Commit message: As built
Parts:
- removed MOD1: ESP12E_DEVKIT, ESP12E_DEVKIT:ESP12E_DEVKIT
- added JP2, JP3: (no value), pinhead:1X15
- moved H2 4.45 mm to (3.17, 92.1)
- moved H3 4.45 mm to (53.3, 92.1)
Connections:
- net A0_SENSOR: now also JP2.1; no longer MOD1.AD0
- net GND: now also JP2.10, JP3.14; no longer MOD1.GND@0, MOD1.GND@3
- net N$2: now also JP2.15; no longer MOD1.VIN
- net RELE_1_IO: now also JP3.4; no longer MOD1.D3
- net RELE_2_IO: now also JP3.5; no longer MOD1.D4
Routing:
- net N$2: track 26.2 -> 27.3 mm
Other:
- board size 160 x 100 mm -> 56.5 x 91.7 mm
