File: sense2.0/Hardware/TBD-board.sch (EAGLE design)
At the start: 17 parts, among them IC1 LM324N, X1 PG203J

Commit message: As built
Parts:
- removed MOD1: ESP12E_DEVKIT, ESP12E_DEVKIT:ESP12E_DEVKIT
- added JP2, JP3: (no value), pinhead:PINHD-1X15
Connections:
- net A0_SENSOR: now also JP2.1; no longer MOD1.AD0
- net GND: now also JP2.10, JP3.14; no longer MOD1.GND@0, MOD1.GND@3
- net N$2: now also JP2.15; no longer MOD1.VIN
- net RELE_1_IO: now also JP3.4; no longer MOD1.D3
- net RELE_2_IO: now also JP3.5; no longer MOD1.D4
Changed lines of the file:
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@@
 <?xml version="1.0" encoding="utf-8"?>
 <!DOCTYPE eagle SYSTEM "eagle.dtd">
-<eagle version="8.3.1">
+<eagle version="8.2.2">
 <drawing>
 <settings>
 <setting alwaysvectorfont="no"/>
-<setting keepoldvectorfont="yes"/>
 <setting verticaltext="up"/>
 </settings>
@@
 </classes>
 <parts>
-<part name="MOD1" library="ESP12E_DEVKIT" deviceset="ESP12E_DEVKIT" device=""/>
 <part name="FONTE" library="hlk-pm01" deviceset="HLK-PM01" device="">
 <attribute name="FONTE" value="127Vac - 5Vcc"/>
@@
 <part name="GND18" library="supply1" deviceset="GND" device=""/>
 <part name="P+2" library="supply1" library_urn="urn:adsk.eagle:library:371" deviceset="+5V" device=""/>
-<part name="X1" library="con-hirschmann" library_urn="urn:adsk.eagle:library:153" deviceset="PG203J" device="" package3d_urn="urn:adsk.eagle:package:7447/1"/>
+<part name="X1" library="con-hirschmann" library_urn="urn:adsk.eagle:library:153" deviceset="PG203J" device=""/>
 <part name="JP1" library="jumper" deviceset="JP1Q" device=""/>
 <part name="C2" library="rcl" deviceset="CPOL-US" device="E2.5-6" value="0.1uF"/>
@@
 <part name="GND2" library="supply1" deviceset="GND" device=""/>
 <part name="P+3" library="supply1" library_urn="urn:adsk.eagle:library:371" deviceset="+5V" device=""/>
-<part name="IC1" library="linear" library_urn="urn:adsk.eagle:library:262" deviceset="LM324" device="N" package3d_urn="urn:adsk.eagle:package:16407/1"/>
-<part name="H1" library="special-drill" library_urn="urn:adsk.eagle:library:366" deviceset="SPECIAL_DRILL_" device="0.1000" package3d_urn="urn:adsk.eagle:package:26539/1"/>
-<part name="H2" library="special-drill" library_urn="urn:adsk.eagle:library:366" deviceset="SPECIAL_DRILL_" device="0.1000" package3d_urn="urn:adsk.eagle:package:26539/1"/>
-<part name="H3" library="special-drill" library_urn="urn:adsk.eagle:library:366" deviceset="SPECIAL_DRILL_" device="0.1000" package3d_urn="urn:adsk.eagle:package:26539/1"/>
-<part name="H4" library="special-drill" library_urn="urn:adsk.eagle:library:366" deviceset="SPECIAL_DRILL_" device="0.1000" package3d_urn="urn:adsk.eagle:package:26539/1"/>
+<part name="IC1" library="linear" library_urn="urn:adsk.eagle:library:262" deviceset="LM324" device="N"/>
+<part name="H1" library="special-drill" library_urn="urn:adsk.eagle:library:366" deviceset="SPECIAL_DRILL_" device="0.1000"/>
+<part name="H2" library="special-drill" library_urn="urn:adsk.eagle:library:366" deviceset="SPECIAL_DRILL_" device="0.1000"/>
+<part name="H3" library="special-drill" library_urn="urn:adsk.eagle:library:366" deviceset="SPECIAL_DRILL_" device="0.1000"/>
+<part name="H4" library="special-drill" library_urn="urn:adsk.eagle:library:366" deviceset="SPECIAL_DRILL_" device="0.1000"/>
+<part name="JP2" library="pinhead" library_urn="urn:adsk.eagle:library:325" deviceset="PINHD-1X15" device=""/>
+<part name="JP3" library="pinhead" library_urn="urn:adsk.eagle:library:325" deviceset="PINHD-1X15" device=""/>
 </parts>
 <sheets>
@@
 </plain>
 <instances>
-<instance part="MOD1" gate="G$1" x="172.72" y="140.97"/>
 <instance part="FONTE" gate="G$1" x="52.07" y="156.21" rot="MR180">
 <attribute name="FONTE" x="59.69" y="161.036" size="1.778" layer="96" rot="MR180"/>
@@
 <instance part="X2" gate="-1" x="44.704" y="156.21"/>
 <instance part="X2" gate="-2" x="44.704" y="151.13"/>
-<instance part="GND5" gate="1" x="199.39" y="125.73" rot="R90"/>
+<instance part="GND5" gate="1" x="199.898" y="125.73" rot="R90"/>
 <instance part="GND7" gate="1" x="257.81" y="107.95"/>
 <instance part="R1" gate="G$1" x="257.81" y="135.89" rot="MR90"/>
@@
 <attribute name="NAME" x="257.302" y="168.656" size="1.778" layer="95"/>
 </instance>
+<instance part="JP2" gate="A" x="157.48" y="140.97"/>
+<instance part="JP3" gate="A" x="187.706" y="140.97" rot="MR0"/>
 </instances>
 <busses>
@@
 </segment>
 <segment>
-<pinref part="MOD1" gate="G$1" pin="GND@3"/>
-<wire x1="190.5" y1="125.73" x2="196.85" y2="125.73" width="0.1524" layer="91"/>
-<pinref part="GND5" gate="1" pin="GND"/>
-</segment>
-<segment>
-<pinref part="MOD1" gate="G$1" pin="GND@0"/>
 <pinref part="GND1" gate="1" pin="GND"/>
 <wire x1="151.13" y1="135.89" x2="154.94" y2="135.89" width="0.1524" layer="91"/>
+<pinref part="JP2" gate="A" pin="10"/>
 </segment>
 <segment>
@@
 <pinref part="IC1" gate="P" pin="V-"/>
 </segment>
+<segment>
+<pinref part="JP3" gate="A" pin="14"/>
+<pinref part="GND5" gate="1" pin="GND"/>
+<wire x1="190.246" y1="125.73" x2="197.358" y2="125.73" width="0.1524" layer="91"/>
+</segment>
 </net>
 <net name="LOAD-" class="0">
@@
 <net name="A0_SENSOR" class="0">
 <segment>
-<pinref part="MOD1" gate="G$1" pin="AD0"/>
-<wire x1="154.94" y1="158.75" x2="153.67" y2="158.75" width="0.1524" layer="91"/>
-<label x="153.67" y="158.75" size="1.778" layer="95" rot="R180" xref="yes"/>
+<wire x1="154.94" y1="158.75" x2="148.336" y2="158.75" width="0.1524" layer="91"/>
+<pinref part="JP2" gate="A" pin="1"/>
+<label x="136.906" y="159.004" size="1.778" layer="95"/>
 </segment>
 <segment>
@@
 <net name="RELE_1_IO" class="0">
 <segment>
-<pinref part="MOD1" gate="G$1" pin="D3"/>
-<wire x1="190.5" y1="151.13" x2="195.58" y2="151.13" width="0.1524" layer="91"/>
+<wire x1="190.246" y1="151.13" x2="196.088" y2="151.13" width="0.1524" layer="91"/>
 <label x="195.58" y="151.13" size="1.778" layer="95"/>
+<pinref part="JP3" gate="A" pin="4"/>
 </segment>
 </net>
 <net name="RELE_2_IO" class="0">
 <segment>
-<pinref part="MOD1" gate="G$1" pin="D4"/>
-<wire x1="190.5" y1="148.59" x2="195.58" y2="148.59" width="0.1524" layer="91"/>
+<wire x1="190.246" y1="148.59" x2="196.088" y2="148.59" width="0.1524" layer="91"/>
 <label x="195.58" y="148.59" size="1.778" layer="95"/>
+<pinref part="JP3" gate="A" pin="5"/>
 </segment>
 </net>
@@
 <net name="N$2" class="0">
 <segment>
-<pinref part="MOD1" gate="G$1" pin="VIN"/>
 <pinref part="JP1" gate="A" pin="1"/>
 <wire x1="150.114" y1="123.19" x2="154.94" y2="123.19" width="0.1524" layer="91"/>
+<pinref part="JP2" gate="A" pin="15"/>
 </segment>
 </net>
@@
 <compatibility>
 <note version="8.2" severity="warning">
-Since Version 8.2, EAGLE supports online libraries. The ids
+Since Version 8.2, Eagle supports online libraries. The ids
 of those online libraries will not be understood (or retained)
 with this version.
 </note>
-<note version="8.3" severity="warning">
-Since Version 8.3, EAGLE supports URNs for individual library
-assets (packages, symbols, and devices). The URNs of those assets
-will not be understood (or retained) with this version.
-</note>
-<note version="8.3" severity="warning">
-Since Version 8.3, EAGLE supports the association of 3D packages
-with devices in libraries, schematics, and board files. Those 3D
-packages will not be understood (or retained) with this version.
-</note>
 </compatibility>
